Commit message: the main issue fixed the odometry calculation issue

File: install/diffdrive_arduino/share/diffdrive_arduino/ros2_control/diffbot.ros2_control.xacro (robot description, xacro)
@@ -1 +1 @@
-/home/ubuntu/robot_ws/src/diffdrive_arduino/description/ros2_control/diffbot.ros2_control.xacro
+/home/ubuntu/dev_Ws/src/diffdrive_arduino/description/ros2_control/diffbot.ros2_control.xacro

File: install/diffdrive_arduino/share/diffdrive_arduino/urdf/diffbot.materials.xacro (robot description, xacro)
@@ -1 +1 @@
-/home/ubuntu/robot_ws/src/diffdrive_arduino/description/urdf/diffbot.materials.xacro
+/home/ubuntu/dev_Ws/src/diffdrive_arduino/description/urdf/diffbot.materials.xacro

File: install/diffdrive_arduino/share/diffdrive_arduino/urdf/diffbot.urdf.xacro (robot description, xacro)
@@ -1 +1 @@
-/home/ubuntu/robot_ws/src/diffdrive_arduino/description/urdf/diffbot.urdf.xacro
+/home/ubuntu/dev_Ws/src/diffdrive_arduino/description/urdf/diffbot.urdf.xacro

File: install/diffdrive_arduino/share/diffdrive_arduino/urdf/diffbot_description.urdf.xacro (robot description, xacro)
@@ -1 +1 @@
-/home/ubuntu/robot_ws/src/diffdrive_arduino/description/urdf/diffbot_description.urdf.xacro
+/home/ubuntu/dev_Ws/src/diffdrive_arduino/description/urdf/diffbot_description.urdf.xacro

File: install/my_bot/share/my_bot/description/gazebo_control.xacro (robot description, xacro)
@@ -1 +1 @@
-/home/ubuntu/robot_ws/src/my_bot/description/gazebo_control.xacro
+/home/ubuntu/dev_Ws/src/my_bot/description/gazebo_control.xacro

File: install/my_bot/share/my_bot/description/inertial_macros.xacro (robot description, xacro)
@@ -1 +1 @@
-/home/ubuntu/robot_ws/src/my_bot/description/inertial_macros.xacro
+/home/ubuntu/dev_Ws/src/my_bot/description/inertial_macros.xacro

File: install/my_bot/share/my_bot/description/lidar.xacro (robot description, xacro)
@@ -1 +1 @@
-/home/ubuntu/robot_ws/src/my_bot/description/lidar.xacro
+/home/ubuntu/dev_Ws/src/my_bot/description/lidar.xacro

File: install/my_bot/share/my_bot/description/robot.urdf.xacro (robot description, xacro)
@@ -1 +1 @@
-/home/ubuntu/robot_ws/src/my_bot/description/robot.urdf.xacro
+/home/ubuntu/dev_Ws/src/my_bot/description/robot.urdf.xacro

File: install/my_bot/share/my_bot/description/robot_core.xacro (robot description, xacro)
@@ -1 +1 @@
-/home/ubuntu/robot_ws/src/my_bot/description/robot_core.xacro
+/home/ubuntu/dev_Ws/src/my_bot/description/robot_core.xacro

File: install/my_bot/share/my_bot/description/ros2_control.xacro (robot description, xacro)
@@ -1 +1 @@
-/home/ubuntu/robot_ws/src/my_bot/description/ros2_control.xacro
+/home/ubuntu/dev_Ws/src/my_bot/description/ros2_control.xacro

File: src/my_bot/description/lidar.xacro (robot description, xacro)
@@ -4,5 +4,5 @@
         <parent link="chassis"/>
         <child link="laser_frame"/>
-        <origin xyz="0.122 0 0.212" rpy="0 0 0"/>
+        <origin xyz="0.22 0 0.212" rpy="0 0 0"/>
     </joint>
     <link name="laser_frame">
@@ -33,5 +33,5 @@
         <sensor name="laser" type="ray">
             <pose> 0 0 0 0 0 0 </pose>
-            <visualize>false</visualize>
+            <visualize>true</visualize>
             <update_rate>10</update_rate>
             <ray>
